Commit message: Added grasp link

File: pose_retargeting/optimization/model/shadowrobot.urdf (robot description, URDF)
Before this commit: robot shadowhand_motor, 33 links, 32 joints
Links:
- added link S_grasp, mass 0.008
Joints:
- added joint grasp_joint: type fixed, parent rh_palm, child S_grasp, origin xyz=.007 -.05 0.07 rpy=0 0 0
